File: led_string.kicad_sch (KiCad schematic)
At the start: 4 parts

Commit message: arrange all components
Parts:
- R1: renamed from R2; value 0.2 -> 1R
Changed lines of the file:
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@@
 		(dnp no)
 		(fields_autoplaced yes)
-		(property "Reference" "R2"
+		(property "Reference" "R1"
 			(at 129.54 91.4399 0)
 			(effects
@@
 			)
 		)
-		(property "Value" "0.2"
+		(property "Value" "1R"
 			(at 129.54 93.9799 0)
 			(effects
@@
 				)
 				(path "/b5279a47-4e53-4efd-ad9f-4a5619d0841f/107d8509-ed25-4b81-a133-c6261c323981"
-					(reference "R2")
+					(reference "R1")
 					(unit 1)
 				)
@@
 				)
 				(path "/b5279a47-4e53-4efd-ad9f-4a5619d0841f/34159603-48d9-4829-b1b4-2af69d99cdd9"
-					(reference "R1")
+					(reference "R2")
 					(unit 1)
 				)
