File: sunface.kicad_pcb (KiCad board)
At the start: 2 copper layers, 128 x 100 mm, 69 parts, among them U1 PT4115

Commit message: finalise design for manufacture
Parts:
- moved Rs1 9.32 mm to (158.0, 95.0), turned to -90 degrees
- moved C1 5.00 mm to (161.0, 95.0), turned to 90 degrees
Routing:
- net Net-(LED8-K): track 0.00 -> 13.7 mm
- net Net-(LED7-K): track 0.00 -> 13.7 mm
- net Net-(LED5-K): track 0.00 -> 13.7 mm
- net Net-(LED47-K): track 0.00 -> 13.7 mm
- net Net-(LED46-K): track 0.00 -> 13.7 mm
- net Net-(LED44-K): track 0.00 -> 13.7 mm
- net Net-(LED43-K): track 0.00 -> 13.7 mm
- net Net-(LED41-K): track 0.00 -> 13.7 mm
- net Net-(LED40-K): track 0.00 -> 13.7 mm
- net Net-(LED4-K): track 0.00 -> 13.7 mm
- net Net-(LED38-K): track 0.00 -> 13.7 mm
- net Net-(LED37-K): track 0.00 -> 13.7 mm
- net Net-(LED35-K): track 0.00 -> 13.7 mm
- net Net-(LED34-K): track 0.00 -> 13.7 mm
- net Net-(LED32-K): track 0.00 -> 13.7 mm
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Other:
- board text added: "12V in"
- board text added: "12V out"
- board text added: "DIM"
- board text added: "GND in"
- board text added: "GND out"
- board text added: "sunface_v0.1 Designed by Ben Green ben@kernowrobotics.co.uk 12/01/2026"
